File: proteusM73tu.kicad_sch (KiCad schematic)
At the start: 16 parts, among them J1 7-967288-1, J2 XH-8A, J3 Conn_01x06, J4 Conn_01x35, J5 Conn_01x35, J6 Conn_01x23, J7 7-967288-1, M1 Module-wbo-0.2, M2 Module-can-0.1, P1 Pad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

Commit message: Progress
Connections:
- net LS1: now also J1.C41
Changed lines of the file:
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@@
   (no_connect (at 245.11 68.58))
   (no_connect (at 302.26 55.88))
+  (wire (pts (xy 36.83 209.55) (xy 50.8 209.55))
+    (stroke (width 0) (type default) (color 0 0 0 0))
+  )
   (wire (pts (xy 118.11 27.94) (xy 152.4 27.94))
     (stroke (width 0) (type solid) (color 0 0 0 0))
@@
   (wire (pts (xy 224.79 48.26) (xy 245.11 48.26))
     (stroke (width 0) (type solid) (color 0 0 0 0))
+  )
+  (wire (pts (xy 224.79 262.89) (xy 245.11 262.89))
+    (stroke (width 0) (type default) (color 0 0 0 0))
+  )
+  (wire (pts (xy 226.06 97.79) (xy 245.11 97.79))
+    (stroke (width 0) (type default) (color 0 0 0 0))
+  )
+  (wire (pts (xy 226.06 100.33) (xy 245.11 100.33))
+    (stroke (width 0) (type default) (color 0 0 0 0))
+  )
+  (wire (pts (xy 226.06 102.87) (xy 245.11 102.87))
+    (stroke (width 0) (type default) (color 0 0 0 0))
   )
   (wire (pts (xy 231.14 212.09) (xy 245.11 212.09))
@@
     (effects (font (size 1.27 1.27)) (justify left bottom))
   )
+  (label "OUT_INJ1" (at 50.8 209.55 0)
+    (effects (font (size 1.27 1.27)) (justify left bottom))
+  )
   (label "HV1" (at 120.65 64.77 180)
     (effects (font (size 1.27 1.27)) (justify right bottom))
@@
     (effects (font (size 1.27 1.27)) (justify left bottom))
   )
+  (label "IN_CLT" (at 224.79 262.89 0)
+    (effects (font (size 1.27 1.27)) (justify left bottom))
+  )
+  (label "OUT_INJ1" (at 226.06 97.79 0)
+    (effects (font (size 1.27 1.27)) (justify left bottom))
+  )

Commit message: PROGRESS
Connections:
- net LS14 is gone; now on net LS START: J4.11 (Pin_11)
- net 12V_MR: now also J1.A8
- net 12V_RAW: now also J1.D26
- net AT4: now also J7.C22
- net GND: now also J1.A4, J1.A6, J1.C21, J1.C50, J7.A4, J7.A6, J7.C47
- net LS10: now also J7.C2
- net LS11: now also J7.C28
- net LS12: now also J7.C27
- net LS13: now also J1.B23
- net LS2: now also J1.C15
- net LS3: now also J1.C40
- net LS4: now also J1.C2
- net LS5: now also J1.C28
- net LS6: now also J1.C27
- net LS7: now also J7.C41
- net LS8: now also J7.C15
- net LS9: now also J7.C40
- net VR1-: now also J1.C13
- net IAT: now reaches J7.C34
- net KNOCK2: now reaches J7.C36
- net SENS_GND: now reaches J7.C37
- net CAM_POS: now reaches J1.C20
- net VR1_POS: now reaches J1.C32
- net KNOCK1: now reaches J1.C49
- net LS START: now reaches J1.D40
- net LS15 renamed LS RAD
- net LS16 renamed LS FUEL
