File: proteusM73tu.kicad_sch (KiCad schematic)
At the start: 16 parts, among them J1 7-967288-1, J2 XH-8A, J3 Conn_01x06, J4 Conn_01x35, J5 Conn_01x35, J6 Conn_01x23, J7 7-967288-1, M1 Module-wbo-0.2, M2 Module-can-0.1, P1 Pad, Q1 ISL9V3040S3S

Commit message: Upd pinout
Parts:
- removed J1, J7: 7-967288-1, lib:79672881, symbol 7-967288-1:7-967288-1
- removed J2: XH-8A, hellen-one-common:XH-8A, symbol Connector_Generic:Conn_01x08
- removed J4: Conn_01x35, lib:ampseal-35, symbol Connector_Generic:Conn_01x35
- removed J5: Conn_01x35, lib:ampseal-35-2, symbol Connector_Generic:Conn_01x35
- removed J6: Conn_01x23, lib:ampseal-23, symbol Connector_Generic:Conn_01x23
- removed M1: Module-wbo-0.2, hellen-one-wbo-0.2:wbo, symbol hellen-one-wbo-0.2:Module-wbo-0.2
- added BRD1: proteus, kicad6-libraries:proteus, symbol proteus:proteus
- added C?: 100n, hellen-one-common:C0603, symbol hellen-one-common:Cap
- added C?: 47p, hellen-one-common:C0603, symbol hellen-one-common:Cap
- added F4: Fuse-Pad-Pad, hellen-one-common:PAD-1206-PAD, symbol hellen-one-common:Fuse-Pad-Pad
- added F5: 10A, hellen-one-common:36911600000, symbol hellen-one-common:Fuse-Pad-Pad
- added J1, J2: Conn_01x02, Connector_Molex:Molex_Mini-Fit_Jr_5569-02A2_2x01_P4.20mm_Horizontal, symbol Connector_Generic:Conn_01x02
- added J10, J7: XH-10AW, Connector_JST:JST_XH_S10B-XH-A_1x10_P2.50mm_Horizontal, symbol Connector_Generic:Conn_01x10
- added J11, J12: XH-10A, Connector_JST:JST_XH_B10B-XH-A_1x10_P2.50mm_Vertical, symbol Connector_Generic:Conn_01x10
- added J13: Conn_01x06, Connector_PinHeader_2.54mm:PinHeader_1x06_P2.54mm_Vertical, symbol Connector_Generic:Conn_01x06
- added J4, J5: XH-6AW, Connector_JST:JST_XH_S6B-XH-A_1x06_P2.50mm_Horizontal, symbol Connector_Generic:Conn_01x06
- added J6: XH-4AW, Connector_JST:JST_XH_S4B-XH-A_1x04_P2.50mm_Horizontal, symbol Connector_Generic:Conn_01x04
- added J8, J9: 7-967288-1, kicad6-libraries:TE_7-967288-1, symbol TE_7-967288-1:7-967288-1
- added M1, M3: Module-wbo-0.3, hellen-one-wbo-0.3:wbo, symbol hellen-one-wbo-0.3:Module-wbo-0.3
- added M4: Module-can-0.1, hellen-one-can-0.1:can, symbol hellen-one-can-0.1:Module-can-0.1
- added P10, P11, P12, P13, P14, P15, P16, P17, P18, P19, P2, P20, P21, P22, P23, P24, P25, P26, P27, P28, P29, P3, P30, P31, P32, P33, P34, P35, P36, P37, P38, P39, P4, P40, P41, P42, P43, P44, P45, P46, P47, P48, P49, P5, P50, P51, P52, P53, P54, P55, P56, P57, P58, P59, P6, P60, P61, P62, P63, P64, P65, P66, P68, P69, P7, P70, P71, P73, P74, P8, P9: Pad, hellen-one-common:PAD-TH, symbol hellen-one-common:Pad
- added Q2: ISL9V3040S3S, Package_TO_SOT_SMD:TO-263-2, symbol Device:Q_NIGBT_GCE
- added R3: 22, hellen-one-common:R0603, symbol hellen-one-common:Res
- added R4: DNP, Resistor_SMD:R_2512_6332Metric, symbol hellen-one-common:Res
- added R?: 51k, hellen-one-common:R0603, symbol hellen-one-common:Res
- added U?: MPXxx6115A, kicad6-libraries:MPX_SOP_SSOP, symbol MPX_SOP_SSOP:MPXxx6115A
Connections:
- net 12V_MR: now also BRD1.B23 (12V_MR), J10.1 (Pin_1), J10.2 (Pin_2), J11.1 (Pin_1), J11.2 (Pin_2), J12.1 (Pin_1), J12.2 (Pin_2), J7.1 (Pin_1), J7.2 (Pin_2)
- net 12V_RAW: now also BRD1.B18 (12V_IGN), F4.2
- net CAN_H: now also BRD1.B17 (CAN+), M4.S2 (CANH)
- net CAN_L: now also BRD1.B16 (CAN-), M4.S1 (CANL)
- net ETB1+: now also BRD1.B7 (ETB1+), J1.2 (Pin_2)
- net ETB1-: now also BRD1.B6 (ETB1-), J1.1 (Pin_1)
- net ETB2+: now also BRD1.B15 (ETB2+), J2.2 (Pin_2)
- net ETB2-: now also BRD1.B8 (ETB2-), J2.1 (Pin_1)
- net GATE_IGN1: now also BRD1.A35 (IGN1)
- net GND: now also BRD1.A17 (GND), BRD1.A18 (GND), BRD1.A24 (GND), BRD1.B14 (GND), BRD1.B19 (GND), BRD1.B20 (GND), BRD1.C1 (GND_SENS), BRD1.C2 (GND_SENS), BRD1.C23 (GND_SENS), BRD1.C29 (GND_SENS), BRD1.C3 (GND_SENS), BRD1.C4 (GND_SENS), BRD1.C5 (GND_SENS), BRD1.C6 (GND_SENS), BRD1.C7 (GND_SENS), BRD1.C8 (GND_SENS), C?.1, C?.1, J10.10 (Pin_10), J10.9 (Pin_9), J11.10 (Pin_10), J11.9 (Pin_9), J12.10 (Pin_10), J12.9 (Pin_9), J13.3 (Pin_3), J4.5 (Pin_5), J4.6 (Pin_6), J5.5 (Pin_5), J5.6 (Pin_6), J6.4 (Pin_4), J7.10 (Pin_10), J7.9 (Pin_9), J8.A4, J8.A6, J8.C19, J8.C37, J8.C45, J8.C47, J8.C50, J8.C6, J8.C9, J8.E1, J9.A4, J9.A6, J9.C21, J9.C37, J9.C45, J9.C50, J9.C6, J9.C9, J9.E1, J9.E5, M1.E6 (LSU_H-), M1.G (GND), M3.E6 (LSU_H-), M3.G (GND), M4.E1 (GND), Q2.3 (E), R?.2, U?.3 (GND)
- net WBO_H-: now also J10.7 (Pin_7), J10.8 (Pin_8), J11.7 (Pin_7), J11.8 (Pin_8), J12.7 (Pin_7), J12.8 (Pin_8), J7.7 (Pin_7), J7.8 (Pin_8), M1.E5 (LSU_H+), M3.E5 (LSU_H+)
- net WBO_Ip: now also J10.5 (Pin_5), J11.5 (Pin_5), J12.5 (Pin_5), J7.5 (Pin_5), M1.E3 (LSU_Ip), M3.E3 (LSU_Ip)
- net WBO_R_Trim: now also J10.6 (Pin_6), J11.6 (Pin_6), J12.6 (Pin_6), J7.6 (Pin_6), M1.E4 (LSU_Rtrim), M3.E4 (LSU_Rtrim)
- net WBO_Vs: now also J10.3 (Pin_3), J11.3 (Pin_3), J12.3 (Pin_3), J7.3 (Pin_3), M1.E1 (LSU_Un), M3.E1 (LSU_Un)
- net WBO_Vs/Ip: now also J10.4 (Pin_4), J11.4 (Pin_4), J12.4 (Pin_4), J7.4 (Pin_4), M1.E2 (LSU_Vm), M3.E2 (LSU_Vm)
- net at M2.V2 (CAN_VIO): now also M3.W2 (CAN_VIO)
- net at M2.V6 (CAN_RX): now also M3.W3 (CAN_RX)
- net at M2.V5 (CAN_TX): now also M3.W4 (CAN_TX)
- net at J3.5 (Pin_5): now also M3.W5 (nReset)
- net at J3.4 (Pin_4): now also M3.W6 (SWDIO)
- net at J3.2 (Pin_2): now also M3.W7 (SWCLK)
- net at J3.1 (Pin_1): now also M3.W8 (V33_OUT)
- net at F1.1: now also J9.A8
- net 5V_SENSOR_2 renamed +5VA
- net +5VA: now also BRD1.C21 (5V_1), BRD1.C32 (5V_1), BRD1.C9 (5V_1), C?.2, J4.1 (Pin_1), J4.2 (Pin_2), J5.1 (Pin_1), J5.2 (Pin_2), J6.1 (Pin_1), M1.W1 (V5_IN), M3.W1 (V5_IN), M4.V1 (V5), U?.2 (Vs)
- new net: J9.B8, P6.1 (Pin_1)
- new net: BRD1.B10 (D1), P59.1 (Pin_1)
- new net: J9.D17, P22.1 (Pin_1)
- new net: M1.J2 (SEL2), M1.J_VCC2 (PULL_UP2)
- new net: M1.W2 (CAN_VIO), M4.V2 (CAN_VIO)
- new net: M1.W3 (CAN_RX), M4.V6 (CAN_RX)
- new net: M1.W4 (CAN_TX), M4.V5 (CAN_TX)
- new net: J13.5 (Pin_5), M1.W5 (nReset)
- new net: J13.4 (Pin_4), M1.W6 (SWDIO)
- new net: J13.2 (Pin_2), M1.W7 (SWCLK)
- new net: J13.1 (Pin_1), M1.W8 (V33_OUT)
- new net: J8.A8, P29.1 (Pin_1)
- new net: J9.B18, P12.1 (Pin_1)
- new net: M3.J1 (SEL1), M3.J_GND1 (PULL_DOWN1)
- new net: J8.C3, P30.1 (Pin_1)
- new net: J9.D36, P26.1 (Pin_1)
- new net: J9.C14, P15.1 (Pin_1)
- new net: J8.C49, P38.1 (Pin_1)
- new net: BRD1.C18 (AV11), P69.1 (Pin_1)
- new net: J9.B15, P10.1 (Pin_1)
- new net: J8.A7, P28.1 (Pin_1)
- new net: J8.C14, P31.1 (Pin_1)
- new net: J8.C18, P32.1 (Pin_1)
- new net: J8.C20, P33.1 (Pin_1)
- new net: J8.C23, P34.1 (Pin_1)
- new net: J8.C32, P35.1 (Pin_1)
- new net: J8.C36, P36.1 (Pin_1)
- new net: J8.C46, P37.1 (Pin_1)
- new net: J8.D10, P40.1 (Pin_1)
- new net: J8.D26, P41.1 (Pin_1)
- new net: J8.D36, P42.1 (Pin_1)
- new net: J8.D37, P43.1 (Pin_1)
- new net: J8.D40, P44.1 (Pin_1)
- new net: J8.D6, P39.1 (Pin_1)
- new net: BRD1.C17 (AV9), P68.1 (Pin_1)
- new net: BRD1.B21 (CAN2-), P66.1 (Pin_1)
- new net: BRD1.A22 (IGN3), P50.1 (Pin_1)
- new net: J9.A7, P2.1 (Pin_1)
- new net: BRD1.C20 (AT3), P71.1 (Pin_1)
- new net: BRD1.C19 (AT1), P70.1 (Pin_1)
- new net: F4.1, J9.D26
- new net: J9.B7, P5.1 (Pin_1)
- new net: BRD1.A32 (IGN5), P52.1 (Pin_1)
- new net: BRD1.A31 (IGN6), P53.1 (Pin_1)
- new net: BRD1.A25 (IGN12), P58.1 (Pin_1)
- new net: BRD1.B9 (D5), P61.1 (Pin_1)
- new net: BRD1.C11 (12V_PROT), P73.1 (Pin_1)
- new net: BRD1.A33 (IGN4), P51.1 (Pin_1)
- new net: BRD1.B12 (VR2-), P64.1 (Pin_1)
- new net: J9.C52, P18.1 (Pin_1)
- new net: Q2.1 (G), R3.1
- new net: BRD1.A13 (HS3), P47.1 (Pin_1)
- new net: J9.C18, P16.1 (Pin_1)
- new net: J9.D37, P27.1 (Pin_1)
- new net: BRD1.A2 (HS1), P45.1 (Pin_1)
- new net: J9.D29, P23.1 (Pin_1)
- new net: BRD1.A1 (HS2), P46.1 (Pin_1)
- new net: BRD1.A14 (HS4), P48.1 (Pin_1)
- new net: BRD1.A26 (IGN11), P57.1 (Pin_1)
- new net: BRD1.A27 (IGN10), P56.1 (Pin_1)
- new net: BRD1.A28 (IGN9), P55.1 (Pin_1)
- new net: BRD1.A29 (IGN8), P54.1 (Pin_1)
- new net: BRD1.A34 (IGN2), P49.1 (Pin_1)
- new net: BRD1.B11 (D6), P62.1 (Pin_1)
- new net: BRD1.B22 (CAN2+), P65.1 (Pin_1)
- new net: BRD1.B3 (D4), P60.1 (Pin_1)
- new net: BRD1.B4 (VR2+), P63.1 (Pin_1)
- new net: BRD1.C12 (12V_PROT), P74.1 (Pin_1)
- new net: J9.D30, P24.1 (Pin_1)
- new net: J9.B9, P7.1 (Pin_1)
- new net: J9.B19, P13.1 (Pin_1)
- new net: J9.B3, P3.1 (Pin_1)
- new net: J9.D34, P25.1 (Pin_1)
- new net: J9.D10, P21.1 (Pin_1)
- new net: J9.C23, P17.1 (Pin_1)
- new net: J9.B17, P11.1 (Pin_1)
- new net: J9.D3, P19.1 (Pin_1)
- new net: J9.B10, P8.1 (Pin_1)
- new net: J9.B11, P9.1 (Pin_1)
- new net: J9.B4, P4.1 (Pin_1)
- new net: J9.C3, P14.1 (Pin_1)
- new net: J9.D6, P20.1 (Pin_1)
- new net GATE_IGN7: BRD1.A30 (IGN7), R3.2, R4.1
- new net HV7: F5.1
- new net IN_BARO: BRD1.C13 (AV1), C?.2, R?.1, U?.4 (Vout)
- new net IN_CAM: BRD1.B1 (D2), J9.C20
- new net IN_CLT: BRD1.C31 (AT4), J9.C22
- new net IN_CRANK+: BRD1.B5 (VR1+), J9.C32
- new net IN_CRANK-: BRD1.B13 (VR1-), J9.C46
- new net IN_IAT: BRD1.C30 (AT2), J8.C34
- new net IN_KNOCK1: BRD1.C34 (KNOCK1), J9.C49
- new net IN_KNOCK2: BRD1.C35 (KNOCK2), J9.C36
- new net IN_PPS1: BRD1.C26 (AV6), J6.2 (Pin_2)
- new net IN_PPS2: BRD1.C16 (AV7), J6.3 (Pin_3)
- new net IN_TPS1_1: BRD1.C24 (AV2), J5.3 (Pin_3)
- new net IN_TPS1_2: BRD1.C14 (AV3), J5.4 (Pin_4)
- new net IN_TPS2_1: BRD1.C25 (AV4), J4.3 (Pin_3)
- new net IN_TPS2_2: BRD1.C15 (AV5), J4.4 (Pin_4)
- new net OUT_IGN7: F5.2, Q2.2 (C), R4.2
- new net OUT_INJ1: BRD1.A3 (LS1), J9.C41
- new net OUT_INJ10: BRD1.A20 (LS10), J8.C2
- new net OUT_INJ11: BRD1.A9 (LS11), J8.C28
- new net OUT_INJ12: BRD1.A21 (LS12), J8.C27
- new net OUT_INJ2: BRD1.A15 (LS2), J9.C15
- new net OUT_INJ3: BRD1.A4 (LS3), J9.C40
- new net OUT_INJ4: BRD1.A16 (LS4), J9.C2
- new net OUT_INJ5: BRD1.A5 (LS5), J9.C28
- new net OUT_INJ6: BRD1.A6 (LS6), J9.C27
- new net OUT_INJ7: BRD1.A7 (LS7), J8.C41
- new net OUT_INJ8: BRD1.A19 (LS8), J8.C15
- new net OUT_INJ9: BRD1.A8 (LS9), J8.C40
- new net OUT_MAIN_RELAY: BRD1.A10 (LS13), J9.B23
- new net OUT_STARTER_EN: BRD1.A11 (LS14), J9.D40
- no-connect marks 5 -> 167
Other:
- note added: "#1"
- note added: "CAN?"
- note added: "TODO: Add "baro" silkscreen"
- note removed: "WHITE"
- moved on the sheet: F1, F3, J3, M2, Q1, R1, R2

Commit message: Upd sch
Parts:
- removed P60, P61: Pad, hellen-one-common:PAD-TH, symbol hellen-one-common:Pad
- added C3: 100n, hellen-one-common:C0603, symbol hellen-one-common:Cap
- added C4: 47p, hellen-one-common:C0603, symbol hellen-one-common:Cap
- added J14, J15: XH-6A, Connector_JST:JST_XH_B6B-XH-A_1x06_P2.50mm_Vertical, symbol Connector_Generic:Conn_01x06
- added J16, J17: XH-6AW, Connector_JST:JST_XH_S6B-XH-A_1x06_P2.50mm_Horizontal, symbol Connector_Generic:Conn_01x06
- added J18: XH-8A, Connector_JST:JST_XH_B8B-XH-A_1x08_P2.50mm_Vertical, symbol Connector_Generic:Conn_01x08
- added J19: XH-8AW, Connector_JST:JST_XH_S8B-XH-A_1x08_P2.50mm_Horizontal, symbol Connector_Generic:Conn_01x08
- added P67: Pad, hellen-one-common:PAD-TH, symbol hellen-one-common:Pad
- added R6: 51k, hellen-one-common:R0603, symbol hellen-one-common:Res
- added U2: MPX4/MPXH6400_MAP, kicad6-libraries:MPX-4_MAP, symbol MPX-4_MAP:MPX4/MPXH6400_MAP
- gave numbers to parts that had none: 4
Connections:
- net +5VA: now also C3.2, J18.1 (Pin_1), J19.1 (Pin_1), U2.3 (VCC)
- net GATE_IGN1: now also J14.1 (Pin_1), J16.1 (Pin_1), P67.1 (Pin_1)
- net GATE_IGN7: now also P68.1 (Pin_1), J15.1 (Pin_1), J17.1 (Pin_1)
- net GND: now also C3.1, C4.1, J18.8 (Pin_8), J19.8 (Pin_8), R6.2, U2.2 (GND)
- net IN_BARO: now also BRD1.C17 (AV9)
- net GATE_IGN3: now reaches BRD1.A22 (IGN3), P50.1 (Pin_1)
- net GATE_IGN3: now also J14.3 (Pin_3), J16.3 (Pin_3)
- net GATE_IGN5: now reaches BRD1.A32 (IGN5), P52.1 (Pin_1)
- net GATE_IGN5: now also J14.5 (Pin_5), J16.5 (Pin_5)
- net GATE_IGN6: now reaches BRD1.A31 (IGN6), P53.1 (Pin_1)
- net GATE_IGN6: now also J14.6 (Pin_6), J16.6 (Pin_6)
- net GATE_IGN12: now reaches BRD1.A25 (IGN12), P58.1 (Pin_1)
- net IN_D5: now reaches BRD1.B9 (D5)
- net IN_D5: now also J18.7 (Pin_7), J19.7 (Pin_7)
- net GATE_IGN4: now reaches BRD1.A33 (IGN4), P51.1 (Pin_1)
- net OUT_FAN_RELAY: now reaches BRD1.A12 (LS15)
- net OUT_FAN_RELAY: now also J18.3 (Pin_3), J19.3 (Pin_3)
- net OUT_FUEL_PUMP: now reaches BRD1.A23 (LS16)
- net OUT_FUEL_PUMP: now also J18.4 (Pin_4), J19.4 (Pin_4)
- net GATE_IGN11: now reaches BRD1.A26 (IGN11), P57.1 (Pin_1)
- net GATE_IGN10: now reaches BRD1.A27 (IGN10), P56.1 (Pin_1)
- net GATE_IGN9: now reaches BRD1.A28 (IGN9), P55.1 (Pin_1)
- net GATE_IGN8: now reaches BRD1.A29 (IGN8), P54.1 (Pin_1)
- net GATE_IGN2: now reaches BRD1.A34 (IGN2), P49.1 (Pin_1)
- net GATE_IGN2: now also J14.2 (Pin_2), J16.2 (Pin_2)
- net IN_START_BTN: now reaches BRD1.B2 (D3)
- net IN_START_BTN: now also J18.5 (Pin_5), J19.5 (Pin_5)
- net IN_D4: now reaches BRD1.B3 (D4)
- net IN_D4: now also J18.6 (Pin_6), J19.6 (Pin_6)
- net IN_MAP: now reaches BRD1.C27 (AV8)
- net IN_MAP: now also C4.2, R6.1, U2.1 (VOUT)
- net IN_AV10: now reaches BRD1.C28 (AV10)
- net IN_AV10: now also J18.2 (Pin_2), J19.2 (Pin_2)
- new net: J15.2 (Pin_2), J17.2 (Pin_2)
- new net: J15.3 (Pin_3), J17.3 (Pin_3)
- new net: J15.4 (Pin_4), J17.4 (Pin_4)
- new net: J15.5 (Pin_5), J17.5 (Pin_5)
- new net: J15.6 (Pin_6), J17.6 (Pin_6)
- new net: J14.4 (Pin_4), J16.4 (Pin_4)
- no-connect marks 167 -> 170
Other:
- note added: "For MPXH6400"
- moved on the sheet: BRD1, C1, C2, F3, F5, J1, J10, J11, J12, J13, J2, J3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

Commit message: Upd SCH
Parts:
- removed F3, F5: 10A, hellen-one-common:36911600000, symbol hellen-one-common:Fuse-Pad-Pad
- removed P17, P34, P69: Pad, hellen-one-common:PAD-TH, symbol hellen-one-common:Pad
- added F? (x6): 10A, hellen-one-common:36911600000, symbol hellen-one-common:Fuse-Pad-Pad
- added G? (x7): PROTO_AREA, hellen-one-common:PROTO_AREA, symbol hellen-one-common:PROTO_AREA
- added P? (x12): Pad, hellen-one-common:PAD-TH, symbol hellen-one-common:Pad
Connections:
- net +5VA: now also G?.10, G?.6, G?.7, G?.8, G?.9
- net GND: now also J8.E5, G?.1, G?.2, G?.3, G?.4, G?.5
- net HV1: now also J9.E3, F?.1
- net IN_BARO: no longer BRD1.C17 (AV9)
- net OUT_IGN1: now also F?.2, F?.2, F?.2
- net OUT_IGN7: now also F?.2, F?.2, F?.2
- net IN_MAF2: now reaches BRD1.C18 (AV11)
- net IN_MAF2: now also J8.C23
- net at J8.B10: now also P?.1 (Pin_1)
- net at J8.B11: now also P?.1 (Pin_1)
- net at J8.B15: now also P?.1 (Pin_1)
- net at J8.B17: now also P?.1 (Pin_1)
- net at J8.B19: now also P?.1 (Pin_1)
- net at J8.B23: now also P?.1 (Pin_1)
- net at J8.B3: now also P?.1 (Pin_1)
- net at J8.B4: now also P?.1 (Pin_1)
- net at J8.B5: now also P?.1 (Pin_1)
- net at J8.B7: now also P?.1 (Pin_1)
- net at J8.B8: now also P?.1 (Pin_1)
- net at J8.B9: now also P?.1 (Pin_1)
- net HV4: now reaches J8.E3
- net HV4: now also F?.1
- net HV5: now reaches J8.E6
- net HV5: now also F?.1
- net HV6: now reaches J8.E9
- net HV6: now also F?.1
- net 12V_PROT: now reaches BRD1.C11 (12V_PROT), P73.1 (Pin_1)
- net 12V_PROT: now also G?.11, G?.12, G?.13, G?.14, G?.15
- net IN_MAF1: now reaches J9.C23
- net IN_MAF1: now also BRD1.C17 (AV9)
- net HV2: now reaches J9.E6
- net HV2: now also F?.1
- net HV3: now reaches J9.E9
- net HV3: now also F?.1
- new net: G?.1, G?.11, G?.6 (x6)
- new net: G?.10, G?.15, G?.5 (x6)
- new net: G?.12, G?.2, G?.7 (x6)
- new net: G?.13, G?.3, G?.8 (x6)
- new net: G?.14, G?.4, G?.9 (x6)
- no-connect marks 170 -> 180
Other:
- moved on the sheet: P73

Commit message: Upd PCB
Parts:
- removed F2: Fuse-Pad-Pad, hellen-one-common:PAD-1206-PAD, symbol hellen-one-common:Fuse-Pad-Pad
- removed F? (x5): 10A, hellen-one-common:36911600000, symbol hellen-one-common:Fuse-Pad-Pad
- removed P1: Pad, hellen-one-common:PAD-TH, symbol hellen-one-common:Pad
- added F3, F5, F6, F7, F8: 10A, kicad6-libraries:FUSE_8.5x4, symbol hellen-one-common:Fuse-Pad-Pad
- F2: renamed from F?; footprint hellen-one-common:36911600000 -> kicad6-libraries:FUSE_8.5x4
- gave numbers to parts that had none: 19
Connections:
- net GATE_IGN1: now also J14.6 (Pin_6), J16.6 (Pin_6); no longer J14.1 (Pin_1), J16.1 (Pin_1)
- net GATE_IGN10: now also J15.3 (Pin_3), J17.3 (Pin_3)
- net GATE_IGN11: now also J15.2 (Pin_2), J17.2 (Pin_2)
- net GATE_IGN12: now also J15.1 (Pin_1), J17.1 (Pin_1)
- net GATE_IGN2: now also J14.5 (Pin_5), J16.5 (Pin_5); no longer J14.2 (Pin_2), J16.2 (Pin_2)
- net GATE_IGN3: now also J14.4 (Pin_4), J16.4 (Pin_4); no longer J14.3 (Pin_3), J16.3 (Pin_3)
- net GATE_IGN4: now also J14.3 (Pin_3), J16.3 (Pin_3)
- net GATE_IGN5: now also J14.2 (Pin_2), J16.2 (Pin_2); no longer J14.5 (Pin_5), J16.5 (Pin_5)
- net GATE_IGN6: now also J14.1 (Pin_1), J16.1 (Pin_1); no longer J14.6 (Pin_6), J16.6 (Pin_6)
- net GATE_IGN7: now also J15.6 (Pin_6), J17.6 (Pin_6); no longer J15.1 (Pin_1), J17.1 (Pin_1)
- net GATE_IGN8: now also J15.5 (Pin_5), J17.5 (Pin_5)
- net GATE_IGN9: now also J15.4 (Pin_4), J17.4 (Pin_4)
- net HV2: now also F3.1
- net HV3: now also F5.1
- net HV4: now also F6.1
- net HV5: now also F7.1
- net HV6: now also F8.1
- net OUT_IGN1: now also F3.2, F5.2
- net OUT_IGN7: now also F6.2, F7.2, F8.2
- net WBO_H-: no longer names the net of J11.7 (Pin_7), J11.8 (Pin_8), J7.7 (Pin_7), J7.8 (Pin_8), M1.E5 (LSU_H+)
- net WBO_H-: no longer J10.7 (Pin_7), J10.8 (Pin_8), J12.7 (Pin_7), J12.8 (Pin_8), M3.E5 (LSU_H+)
- net WBO_Ip: no longer names the net of J11.5 (Pin_5), J7.5 (Pin_5), M1.E3 (LSU_Ip)
- net WBO_Ip: no longer J10.5 (Pin_5), J12.5 (Pin_5), M3.E3 (LSU_Ip)
- net WBO_R_Trim: no longer names the net of J11.6 (Pin_6), J7.6 (Pin_6), M1.E4 (LSU_Rtrim)
- net WBO_R_Trim: no longer J10.6 (Pin_6), J12.6 (Pin_6), M3.E4 (LSU_Rtrim)
- net WBO_Vs: no longer names the net of J11.3 (Pin_3), J7.3 (Pin_3), M1.E1 (LSU_Un)
- net WBO_Vs: no longer J10.3 (Pin_3), J12.3 (Pin_3), M3.E1 (LSU_Un)
- net WBO_Vs/Ip: no longer names the net of J11.4 (Pin_4), J7.4 (Pin_4), M1.E2 (LSU_Vm)
- net WBO_Vs/Ip: no longer J10.4 (Pin_4), J12.4 (Pin_4), M3.E2 (LSU_Vm)
- new net: J10.3 (Pin_3), J12.3 (Pin_3), M3.E1 (LSU_Un)
- new net: J10.4 (Pin_4), J12.4 (Pin_4), M3.E2 (LSU_Vm)
- new net: J10.5 (Pin_5), J12.5 (Pin_5), M3.E3 (LSU_Ip)
- new net: J10.6 (Pin_6), J12.6 (Pin_6), M3.E4 (LSU_Rtrim)
- new net: J10.7 (Pin_7), J10.8 (Pin_8), J12.7 (Pin_7), J12.8 (Pin_8), M3.E5 (LSU_H+)
Other:
- note removed: "Example"
- moved on the sheet: J14, J15, J16, J17

Commit message: Fab preview
Parts:
- added J20: Conn_01x01, TestPoint:TestPoint_Pad_D2.0mm, symbol Connector_Generic:Conn_01x01
- J19: LCSC XH-8AW -> C10395
Connections:
- net GND: now also J20.1 (Pin_1)
- net IN_TPS1_1: now also J4.3 (Pin_3); no longer J5.3 (Pin_3)
- net IN_TPS1_2: now also J4.4 (Pin_4); no longer J5.4 (Pin_4)
- net IN_TPS2_1: now also J5.3 (Pin_3); no longer J4.3 (Pin_3)
- net IN_TPS2_2: now also J5.4 (Pin_4); no longer J4.4 (Pin_4)
- net ETB1+ renamed ETB+1
- net ETB+1: now also J2.2 (Pin_2); no longer J1.2 (Pin_2)
- net ETB1- renamed ETB-1
- net ETB-1: now also J2.1 (Pin_1); no longer J1.1 (Pin_1)
- net ETB2+ renamed ETB+2
- net ETB+2: now also J1.2 (Pin_2); no longer J2.2 (Pin_2)
- net ETB2- renamed ETB-2
- net ETB-2: now also J1.1 (Pin_1); no longer J2.1 (Pin_1)
Other:
- moved on the sheet: J1, J10, J11, J12, J13, J2, J3, J4, J5, J6, J7, M1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
