File: proteusM73tu.kicad_pcb (KiCad board)
At the start: 2 copper layers, 288 x 129 mm, 16 parts, among them J1 7-967288-1, J2 XH-8A, J3 Conn_01x06, J4 Conn_01x35, J5 Conn_01x35, J6 Conn_01x23, J7 7-967288-1, M1 Module-wbo-0.2, M2 Module-can-0.1, P1 Pad, Q1 ISL9V3040S3S

Commit message: Upd pinout
Parts:
- added BRD1: proteus, kicad6-libraries:proteus, F.Cu at (206.6, 116.0)
- added F4: Fuse-Pad-Pad, hellen-one-common:PAD-1206-PAD, F.Cu at (501.3, 131.1)
- added F5: 10A, hellen-one-common:36911600000, F.Cu at (448.5, 172.7)
- added J10: XH-10AW, Connector_JST:JST_XH_S10B-XH-A_1x10_P2.50mm_Horizontal, F.Cu at (439.6, 132.7)
- added J13: Conn_01x06, Connector_PinHeader_2.54mm:PinHeader_1x06_P2.54mm_Vertical, F.Cu at (494.8, 131.7)
- added J8: 7-967288-1, kicad6-libraries:TE_7-967288-1, F.Cu at (139.2, 96.9)
- added J9: 7-967288-1, kicad6-libraries:TE_7-967288-1, F.Cu at (309.2, 96.9)
- added M3: Module-wbo-0.3, hellen-one-wbo-0.3:wbo, F.Cu at (462.4, 75.3)
- added M4: Module-can-0.1, hellen-one-can-0.1:can, F.Cu at (473.8, 150.6)
- added P10: Pad, hellen-one-common:PAD-TH, F.Cu at (507.3, 131.3)
- added P11: Pad, hellen-one-common:PAD-TH, F.Cu at (506.5, 150.2)
- added P12: Pad, hellen-one-common:PAD-TH, F.Cu at (500.3, 161.1)
- added P13: Pad, hellen-one-common:PAD-TH, F.Cu at (496.5, 153.6)
- added P14: Pad, hellen-one-common:PAD-TH, F.Cu at (521.7, 135.1)
- added P15: Pad, hellen-one-common:PAD-TH, F.Cu at (485.2, 153.2)
- added P16: Pad, hellen-one-common:PAD-TH, F.Cu at (499.1, 146.0)
- added P17: Pad, hellen-one-common:PAD-TH, F.Cu at (496.5, 157.3)
- added P18: Pad, hellen-one-common:PAD-TH, F.Cu at (495.1, 148.7)
- added P19: Pad, hellen-one-common:PAD-TH, F.Cu at (487.0, 168.3)
- added P2: Pad, hellen-one-common:PAD-TH, F.Cu at (487.6, 148.7)
- added P20: Pad, hellen-one-common:PAD-TH, F.Cu at (487.0, 172.1)
- added P21: Pad, hellen-one-common:PAD-TH, F.Cu at (500.3, 153.6)
- added P22: Pad, hellen-one-common:PAD-TH, F.Cu at (522.4, 131.3)
- added P23: Pad, hellen-one-common:PAD-TH, F.Cu at (510.4, 135.1)
- added P24: Pad, hellen-one-common:PAD-TH, F.Cu at (498.9, 149.8)
- added P25: Pad, hellen-one-common:PAD-TH, F.Cu at (479.4, 174.5)
- added P26: Pad, hellen-one-common:PAD-TH, F.Cu at (455.2, 172.0)
- added P27: Pad, hellen-one-common:PAD-TH, F.Cu at (479.4, 167.0)
- added P28: Pad, hellen-one-common:PAD-TH, F.Cu at (485.2, 164.5)
- added P29: Pad, hellen-one-common:PAD-TH, F.Cu at (518.0, 138.9)
- added P3: Pad, hellen-one-common:PAD-TH, F.Cu at (489.0, 163.8)
- added P30: Pad, hellen-one-common:PAD-TH, F.Cu at (504.1, 154.0)
- added P31: Pad, hellen-one-common:PAD-TH, F.Cu at (510.3, 150.2)
- added P32: Pad, hellen-one-common:PAD-TH, F.Cu at (496.5, 161.1)
- added P33: Pad, hellen-one-common:PAD-TH, F.Cu at (502.8, 146.0)
- added P34: Pad, hellen-one-common:PAD-TH, F.Cu at (510.4, 146.4)
- added P35: Pad, hellen-one-common:PAD-TH, F.Cu at (489.0, 152.4)
- added P36: Pad, hellen-one-common:PAD-TH, F.Cu at (526.2, 131.3)
- added P37: Pad, hellen-one-common:PAD-TH, F.Cu at (506.6, 138.9)
- added P38: Pad, hellen-one-common:PAD-TH, F.Cu at (459.0, 172.0)
- added P39: Pad, hellen-one-common:PAD-TH, F.Cu at (499.1, 134.7)
- added P4: Pad, hellen-one-common:PAD-TH, F.Cu at (514.2, 142.7)
- added P40: Pad, hellen-one-common:PAD-TH, F.Cu at (506.6, 146.4)
- added P41: Pad, hellen-one-common:PAD-TH, F.Cu at (489.0, 156.2)
- added P42: Pad, hellen-one-common:PAD-TH, F.Cu at (492.8, 160.0)
- added P43: Pad, hellen-one-common:PAD-TH, F.Cu at (490.8, 167.6)
- added P44: Pad, hellen-one-common:PAD-TH, F.Cu at (510.4, 138.9)
- added P45: Pad, hellen-one-common:PAD-TH, F.Cu at (485.2, 160.8)
- added P46: Pad, hellen-one-common:PAD-TH, F.Cu at (514.2, 135.1)
- added P47: Pad, hellen-one-common:PAD-TH, F.Cu at (502.8, 142.2)
- added P48: Pad, hellen-one-common:PAD-TH, F.Cu at (502.7, 149.8)
- added P49: Pad, hellen-one-common:PAD-TH, F.Cu at (514.9, 131.3)
- added P5: Pad, hellen-one-common:PAD-TH, F.Cu at (458.0, 179.5)
- added P50: Pad, hellen-one-common:PAD-TH, F.Cu at (487.6, 144.9)
- added P51: Pad, hellen-one-common:PAD-TH, F.Cu at (485.2, 157.0)
- added P52: Pad, hellen-one-common:PAD-TH, F.Cu at (511.1, 131.3)
- added P53: Pad, hellen-one-common:PAD-TH, F.Cu at (502.8, 138.4)
- added P54: Pad, hellen-one-common:PAD-TH, F.Cu at (489.0, 160.0)
- added P55: Pad, hellen-one-common:PAD-TH, F.Cu at (492.8, 163.8)
- added P56: Pad, hellen-one-common:PAD-TH, F.Cu at (479.4, 178.3)
- added P57: Pad, hellen-one-common:PAD-TH, F.Cu at (483.2, 175.9)
- added P58: Pad, hellen-one-common:PAD-TH, F.Cu at (499.1, 142.2)
- added P59: Pad, hellen-one-common:PAD-TH, F.Cu at (518.0, 135.1)
- added P6: Pad, hellen-one-common:PAD-TH, F.Cu at (514.2, 138.9)
- added P60: Pad, hellen-one-common:PAD-TH, F.Cu at (500.3, 157.3)
- added P61: Pad, hellen-one-common:PAD-TH, F.Cu at (491.4, 148.7)
- added P62: Pad, hellen-one-common:PAD-TH, F.Cu at (483.2, 168.3)
- added P63: Pad, hellen-one-common:PAD-TH, F.Cu at (492.8, 156.2)
- added P64: Pad, hellen-one-common:PAD-TH, F.Cu at (492.8, 152.4)
- added P65: Pad, hellen-one-common:PAD-TH, F.Cu at (479.4, 170.7)
- added P66: Pad, hellen-one-common:PAD-TH, F.Cu at (454.2, 179.5)
- added P67: Pad, hellen-one-common:PAD-TH, F.Cu at (483.2, 172.1)
- added P68: Pad, hellen-one-common:PAD-TH, F.Cu at (459.0, 175.7)
- added P69: Pad, hellen-one-common:PAD-TH, F.Cu at (455.2, 175.7)
- added P7: Pad, hellen-one-common:PAD-TH, F.Cu at (506.6, 142.7)
- added P70: Pad, hellen-one-common:PAD-TH, F.Cu at (499.1, 138.4)
- added P71: Pad, hellen-one-common:PAD-TH, F.Cu at (502.8, 134.7)
- added P72: Pad, hellen-one-common:PAD-TH, F.Cu at (510.4, 142.7)
- added P73: Pad, hellen-one-common:PAD-TH, F.Cu at (506.6, 135.1)
- added P74: Pad, hellen-one-common:PAD-TH, F.Cu at (518.7, 131.3)
- added P8: Pad, hellen-one-common:PAD-TH, F.Cu at (514.2, 146.4)
- added P9: Pad, hellen-one-common:PAD-TH, F.Cu at (496.5, 164.9)
- added Q2: ISL9V3040S3S, Package_TO_SOT_SMD:TO-263-2, F.Cu at (474.5, 158.9)
- added R3: 22, hellen-one-common:R0603, F.Cu at (437.8, 180.8)
- added R4: DNP, Resistor_SMD:R_2512_6332Metric, F.Cu at (448.0, 177.7)
- J1: value 7-967288-1 -> Conn_01x02; footprint lib:79672881 -> Connector_Molex:Molex_Mini-Fit_Jr_5569-02A2_2x01_P4.20mm_Horizontal
- J2: value XH-8A -> Conn_01x02; footprint hellen-one-common:XH-8A -> Connector_Molex:Molex_Mini-Fit_Jr_5569-02A2_2x01_P4.20mm_Horizontal
- J4: value Conn_01x35 -> XH-6AW; footprint lib:ampseal-35 -> Connector_JST:JST_XH_S6B-XH-A_1x06_P2.50mm_Horizontal
- J5: value Conn_01x35 -> XH-6AW; footprint lib:ampseal-35-2 -> Connector_JST:JST_XH_S6B-XH-A_1x06_P2.50mm_Horizontal
- J6: value Conn_01x23 -> XH-4AW; footprint lib:ampseal-23 -> Connector_JST:JST_XH_S4B-XH-A_1x04_P2.50mm_Horizontal
- J7: value 7-967288-1 -> XH-10AW; footprint lib:79672881 -> Connector_JST:JST_XH_S10B-XH-A_1x10_P2.50mm_Horizontal
- M1: value Module-wbo-0.2 -> Module-wbo-0.3; footprint hellen-one-wbo-0.2:wbo -> hellen-one-wbo-0.3:wbo
- moved M2 597.5 mm to (868.0, 61.2)
- moved R1 597.5 mm to (873.3, 62.9)
- moved F1 597.5 mm to (821.3, 71.6)
- moved F2 597.5 mm to (813.0, 71.6)
- moved F3 597.5 mm to (854.4, 68.5)
- moved J3 597.5 mm to (793.3, 42.0)
- moved P1 597.5 mm to (869.8, 63.8)
- moved Q1 597.5 mm to (858.4, 59.7)
- moved R2 597.5 mm to (863.6, 68.4)
- moved J4 335.7 mm to (476.5, 132.7)
- moved M1 263.7 mm to (462.4, 59.0)
- moved J7 257.7 mm to (421.9, 126.7), turned to 0 degrees
- moved J2 257.0 mm to (469.3, 144.3)
- moved J6 86.8 mm to (311.4, 172.6)
- moved J1 82.9 mm to (275.3, 171.1)
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Connections:
- F1 pad 1: unconnected-(F1-Pad1) -> Net-(F1-Pad1)
- J2 pad 1: GND -> /ETB2-
- J2 pad 2: GND -> /ETB2+
- J4 pad 1: (no net) -> +5VA
- J4 pad 2: (no net) -> +5VA
- J4 pad 3: /LS1 -> (no net)
- J4 pad 4: /LS3 -> (no net)
- J4 pad 5: /LS5 -> GND
- J4 pad 6: /LS6 -> GND
- J5 pad 1: GND -> +5VA
- J5 pad 2: GND -> +5VA
- J5 pad 3: GND -> (no net)
- J5 pad 4: GND -> (no net)
- J6 pad 1: /DIGITAL_2 -> +5VA
- J6 pad 2: /DIGITAL_3 -> (no net)
- J6 pad 3: /DIGITAL_4 -> (no net)
- J6 pad 4: (no net) -> GND
- M1 pad J1: Net-(M1-PadJ1) -> (no net)
- M1 pad J2: (no net) -> Net-(M1-PadJ2)
- M1 pad J_GND1: Net-(M1-PadJ1) -> (no net)
- M1 pad J_VCC2: (no net) -> Net-(M1-PadJ2)
- M1 pad W2: Net-(M1-PadW2) -> Net-(M4-PadV2)
- M1 pad W3: Net-(M1-PadW3) -> Net-(M4-PadV6)
- M1 pad W4: Net-(M1-PadW4) -> Net-(M4-PadV5)
- M1 pad W5: Net-(J3-Pad5) -> Net-(J13-Pad5)
- M1 pad W6: Net-(J3-Pad4) -> Net-(J13-Pad4)
- M1 pad W7: Net-(J3-Pad2) -> Net-(J13-Pad2)
- M1 pad W8: Net-(J3-Pad1) -> Net-(J13-Pad1)
- M2 pad S1: (no net) -> /CAN_L
- M2 pad S2: (no net) -> /CAN_H
- M2 pad V2: Net-(M1-PadW2) -> Net-(M2-PadV2)
- M2 pad V5: Net-(M1-PadW4) -> Net-(M2-PadV5)
- M2 pad V6: Net-(M1-PadW3) -> Net-(M2-PadV6)
Other:
- board size 288 x 129 mm -> 334 x 118 mm
- board text added: "BLACK"
- board text added: "GRAY"

Commit message: Upd sch
Parts:
- removed P60, P61, P72: Pad, hellen-one-common:PAD-TH
- added C1: 100n, hellen-one-common:C0603, F.Cu at (512.3, -28.1)
- added C2: 47p, hellen-one-common:C0603, F.Cu at (511.7, -24.9)
- added C3: 100n, hellen-one-common:C0603, F.Cu at (485.5, -15.6)
- added C4: 47p, hellen-one-common:C0603, F.Cu at (481.3, 3.40)
- added J16: XH-6AW, Connector_JST:JST_XH_S6B-XH-A_1x06_P2.50mm_Horizontal, F.Cu at (533.0, 166.2)
- added J17: XH-6AW, Connector_JST:JST_XH_S6B-XH-A_1x06_P2.50mm_Horizontal, F.Cu at (557.5, 152.6)
- added J19: XH-8AW, Connector_JST:JST_XH_S8B-XH-A_1x08_P2.50mm_Horizontal, F.Cu at (533.0, 152.6)
- added R5: 51k, hellen-one-common:R0603, F.Cu at (509.8, -24.8)
- added R6: 51k, hellen-one-common:R0603, F.Cu at (481.1, 6.93)
- added U1: MPXxx6115A, kicad6-libraries:MPX_SOP_SSOP, F.Cu at (523.9, -28.2)
- added U2: MPX4/MPXH6400_MAP, kicad6-libraries:MPX-4_MAP, F.Cu at (489.3, -35.3)
- moved P68 72.5 mm to (531.4, 178.3)
- moved P67 68.1 mm to (550.9, 164.8)
Connections:
- net Net-(BRD1-PadA22) renamed /GATE_IGN3
- net Net-(BRD1-PadA25) renamed /GATE_IGN12
- net Net-(BRD1-PadA26) renamed /GATE_IGN11
- net Net-(BRD1-PadA27) renamed /GATE_IGN10
- net Net-(BRD1-PadA28) renamed /GATE_IGN9
- net Net-(BRD1-PadA29) renamed /GATE_IGN8
- net Net-(BRD1-PadA31) renamed /GATE_IGN6
- net Net-(BRD1-PadA32) renamed /GATE_IGN5
- net Net-(BRD1-PadA33) renamed /GATE_IGN4
- net Net-(BRD1-PadA34) renamed /GATE_IGN2
- BRD1 pad A12: (no net) -> /OUT_FAN_RELAY
- BRD1 pad A23: (no net) -> /OUT_FUEL_PUMP
- BRD1 pad B2: (no net) -> /IN_START_BTN
- BRD1 pad B3: Net-(BRD1-PadB3) -> /IN_D4
- BRD1 pad B9: Net-(BRD1-PadB9) -> /IN_D5
- BRD1 pad C13: Net-(BRD1-PadC13) -> /IN_BARO
- BRD1 pad C14: (no net) -> /IN_TPS1_2
- BRD1 pad C15: (no net) -> /IN_TPS2_2
- BRD1 pad C16: (no net) -> /IN_PPS2
- BRD1 pad C17: Net-(BRD1-PadC17) -> /IN_BARO
- BRD1 pad C21: (no net) -> +5VA
- BRD1 pad C24: (no net) -> /IN_TPS1_1
- BRD1 pad C25: (no net) -> /IN_TPS2_1
- BRD1 pad C26: (no net) -> /IN_PPS1
- BRD1 pad C27: (no net) -> /IN_MAP
- BRD1 pad C28: (no net) -> /IN_AV10
- BRD1 pad C32: (no net) -> +5VA
- BRD1 pad C33: Net-(BRD1-PadC33) -> (no net)
- BRD1 pad C9: (no net) -> +5VA
- J4 pad 3: (no net) -> /IN_TPS2_1
- J4 pad 4: (no net) -> /IN_TPS2_2
- J5 pad 3: (no net) -> /IN_TPS1_1
- J5 pad 4: (no net) -> /IN_TPS1_2
- J6 pad 2: (no net) -> /IN_PPS1
- J6 pad 3: (no net) -> /IN_PPS2
- M1 pad W1: /5V_SENSOR_2 -> +5VA
- M2 pad V1: /5V_SENSOR_2 -> +5VA
- M3 pad W1: /5V_SENSOR_2 -> +5VA
- M4 pad V1: /5V_SENSOR_2 -> +5VA
- P67 pad 1: Net-(BRD1-PadC13) -> /GATE_IGN1
- P68 pad 1: Net-(BRD1-PadC17) -> /GATE_IGN7
Other:
- board text added: "BARO"

Commit message: Upd SCH
Parts:
- added G***: LOGO, LOGO, F.Cu at (272.4, 177.4)
- moved J1 35.3 mm to (282.9, 136.6)
- moved J5 35.3 mm to (295.4, 138.2)
- moved J6 35.3 mm to (318.9, 138.1)
Other:
- board text added: "Proteus BMW M73tu adapter rev. a"
- board text added: "https://rusefi.com/s/proteus-M73tu"
