File: proteusM73tu.kicad_pcb (KiCad board)
At the start: 2 copper layers, 334 x 118 mm, 110 parts, among them J1 Conn_01x02, J10 XH-10AW, J13 Conn_01x06, J16 XH-6AW, J17 XH-6AW, J19 XH-8AW, J2 Conn_01x02, J3 Conn_01x06, J4 XH-6AW, J5 XH-6AW, J6 XH-4AW, J7 XH-10AW, J8 7-967288-1, J9 7-967288-1, M1 Module-wbo-0.3, M2 Module-can-0.1, M3 Module-wbo-0.3, M4 Module-can-0.1, P1 Pad, P10 Pad, P11 Pad, P12 Pad, P13 Pad, P14 Pad, P15 Pad, P16 Pad, P17 Pad, P18 Pad, P19 Pad, P2 Pad, P20 Pad, P21 Pad, P22 Pad, P23 Pad, P24 Pad, P25 Pad, P26 Pad, P27 Pad, P28 Pad, P29 Pad, P3 Pad, P30 Pad, P31 Pad, P32 Pad, P33 Pad, P34 Pad, P35 Pad, P36 Pad, P37 Pad, P38 Pad, P39 Pad, P4 Pad, P40 Pad, P41 Pad, P42 Pad, P43 Pad, P44 Pad, P45 Pad, P46 Pad, P47 Pad, P48 Pad, P49 Pad, P5 Pad, P50 Pad, P51 Pad, P52 Pad, P53 Pad, P54 Pad, P55 Pad, P56 Pad, P57 Pad, P58 Pad, P59 Pad, P6 Pad, P62 Pad, P63 Pad, P64 Pad, P65 Pad, P66 Pad, P67 Pad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

Commit message: Upd PCB
Parts:
- added F6: 10A, kicad6-libraries:FUSE_8.5x4, F.Cu at (72.5, 140.8)
- added F7: 10A, kicad6-libraries:FUSE_8.5x4, F.Cu at (78.0, 140.8)
- added F8: 10A, kicad6-libraries:FUSE_8.5x4, F.Cu at (83.4, 140.8)
- added G1: PROTO_AREA, hellen-one-common:PROTO_AREA, F.Cu at (126.4, 184.8)
- added G2: PROTO_AREA, hellen-one-common:PROTO_AREA, F.Cu at (118.8, 172.1)
- added G3: PROTO_AREA, hellen-one-common:PROTO_AREA, F.Cu at (126.4, 172.1)
- added G4: PROTO_AREA, hellen-one-common:PROTO_AREA, F.Cu at (111.2, 184.8)
- added G5: PROTO_AREA, hellen-one-common:PROTO_AREA, F.Cu at (126.4, 192.4)
- added G6: PROTO_AREA, hellen-one-common:PROTO_AREA, F.Cu at (118.8, 184.8)
- added G7: PROTO_AREA, hellen-one-common:PROTO_AREA, F.Cu at (111.2, 172.1)
- added P60: Pad, hellen-one-common:PAD-TH, F.Cu at (185.0, 137.8)
- added P61: Pad, hellen-one-common:PAD-TH, F.Cu at (181.5, 137.8)
- added P72: Pad, hellen-one-common:PAD-TH, F.Cu at (170.5, 147.3)
- added P75: Pad, hellen-one-common:PAD-TH, F.Cu at (161.5, 139.8)
- added P76: Pad, hellen-one-common:PAD-TH, F.Cu at (174.0, 139.8)
- added P77: Pad, hellen-one-common:PAD-TH, F.Cu at (164.5, 144.3)
- added P78: Pad, hellen-one-common:PAD-TH, F.Cu at (178.0, 137.8)
- added P79: Pad, hellen-one-common:PAD-TH, F.Cu at (164.5, 139.8)
- F2: value Fuse-Pad-Pad -> 10A; footprint hellen-one-common:PAD-1206-PAD -> kicad6-libraries:FUSE_8.5x4
- F3, F5: footprint hellen-one-common:36911600000 -> kicad6-libraries:FUSE_8.5x4
- Q1, R1, R2: moved to B.Cu
- moved P1 701.0 mm to (174.0, 148.8)
- moved R1 666.2 mm to (213.3, 153.1)
- moved Q1 658.2 mm to (205.8, 145.6), turned to 90 degrees
- moved R2 654.6 mm to (213.8, 148.1), turned to 90 degrees
- moved F3 647.1 mm to (210.0, 127.5), turned to 180 degrees
- moved F2 605.2 mm to (210.0, 123.1), turned to 180 degrees
- moved M2 560.7 mm to (315.1, 154.5), turned to -90 degrees
- moved F1 494.5 mm to (331.5, 139.8), turned to -90 degrees
- moved J19 487.5 mm to (46.5, 183.3), turned to -90 degrees
- moved J3 478.1 mm to (333.2, 172.1), turned to -90 degrees
- moved U2 477.7 mm to (78.5, 208.5), turned to 180 degrees
- moved C1 473.8 mm to (98.5, 202.6)
- moved C2 473.8 mm to (97.9, 205.8)
- moved R5 473.8 mm to (95.9, 205.9)
- moved U1 473.8 mm to (110.0, 202.6)
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Connections:
- net Net-(BRD1-PadC11) renamed /12V_PROT
- BRD1 pad C17: /IN_BARO -> /IN_MAF1
- BRD1 pad C18: Net-(BRD1-PadC18) -> /IN_MAF2
- F2 pad 1: unconnected-(F2-Pad1) -> /HV1
- F2 pad 2: /12V_MR -> /OUT_IGN1
- F3 pad 1: (no net) -> /HV2
- F5 pad 1: (no net) -> /HV3
- F5 pad 2: /OUT_IGN7 -> /OUT_IGN1
- J10 pad 3: /WBO_Vs -> Net-(J10-Pad3)
- J10 pad 4: /WBO_Vs/Ip -> Net-(J10-Pad4)
- J10 pad 5: /WBO_Ip -> Net-(J10-Pad5)
- J10 pad 6: /WBO_R_Trim -> Net-(J10-Pad6)
- J10 pad 7: /WBO_H- -> Net-(J10-Pad7)
- J10 pad 8: /WBO_H- -> Net-(J10-Pad7)
- J16 pad 1: /GATE_IGN1 -> /GATE_IGN6
- J16 pad 2: /GATE_IGN2 -> /GATE_IGN5
- J16 pad 3: /GATE_IGN3 -> /GATE_IGN4
- J16 pad 4: (no net) -> /GATE_IGN3
- J16 pad 5: /GATE_IGN5 -> /GATE_IGN2
- J16 pad 6: /GATE_IGN6 -> /GATE_IGN1
- J17 pad 1: /GATE_IGN7 -> /GATE_IGN12
- J17 pad 2: (no net) -> /GATE_IGN11
- J17 pad 3: (no net) -> /GATE_IGN10
- J17 pad 4: (no net) -> /GATE_IGN9
- J17 pad 5: (no net) -> /GATE_IGN8
- J17 pad 6: (no net) -> /GATE_IGN7
- J7 pad 3: /WBO_Vs -> Net-(J11-Pad3)
- J7 pad 4: /WBO_Vs/Ip -> Net-(J11-Pad4)
- J7 pad 5: /WBO_Ip -> Net-(J11-Pad5)
- J7 pad 6: /WBO_R_Trim -> Net-(J11-Pad6)
- J7 pad 7: /WBO_H- -> Net-(J11-Pad7)
- J7 pad 8: /WBO_H- -> Net-(J11-Pad7)
- J8 pad B10: (no net) -> Net-(J8-PadB10)
- J8 pad B11: (no net) -> Net-(J8-PadB11)
- J8 pad B15: (no net) -> Net-(J8-PadB15)
- J8 pad B17: (no net) -> Net-(J8-PadB17)
- J8 pad B19: (no net) -> Net-(J8-PadB19)
- J8 pad B23: (no net) -> Net-(J8-PadB23)
- J8 pad B3: (no net) -> Net-(J8-PadB3)
- J8 pad B4: (no net) -> Net-(J8-PadB4)
- J8 pad B5: (no net) -> Net-(J8-PadB5)
- J8 pad B7: (no net) -> Net-(J8-PadB7)
- J8 pad B8: (no net) -> Net-(J8-PadB8)
- J8 pad B9: (no net) -> Net-(J8-PadB9)
- J8 pad C23: Net-(J8-PadC23) -> /IN_MAF2
- J8 pad E3: (no net) -> /HV4
- J8 pad E5: (no net) -> GND
- J8 pad E6: (no net) -> /HV5
- J8 pad E9: (no net) -> /HV6
- J9 pad C23: Net-(J9-PadC23) -> /IN_MAF1
- J9 pad E3: (no net) -> /HV1
- J9 pad E6: (no net) -> /HV2
- J9 pad E9: (no net) -> /HV3
- M1 pad E1: /WBO_Vs -> Net-(J11-Pad3)
- M1 pad E2: /WBO_Vs/Ip -> Net-(J11-Pad4)
- M1 pad E3: /WBO_Ip -> Net-(J11-Pad5)
- M1 pad E4: /WBO_R_Trim -> Net-(J11-Pad6)
- M1 pad E5: /WBO_H- -> Net-(J11-Pad7)
- M3 pad E1: /WBO_Vs -> Net-(J10-Pad3)
- M3 pad E2: /WBO_Vs/Ip -> Net-(J10-Pad4)
- M3 pad E3: /WBO_Ip -> Net-(J10-Pad5)
- M3 pad E4: /WBO_R_Trim -> Net-(J10-Pad6)
- M3 pad E5: /WBO_H- -> Net-(J10-Pad7)
- P1 pad 1: (no net) -> Net-(J8-PadB3)
- P17 pad 1: Net-(J9-PadC23) -> Net-(J8-PadB4)
- P34 pad 1: Net-(J8-PadC23) -> Net-(J8-PadB5)
- P69 pad 1: Net-(BRD1-PadC18) -> Net-(J8-PadB9)
Routing:
- net +5VA: track 0.00 -> 283.7 mm, vias 0 -> 6
- net /OUT_FAN_RELAY: track 0.00 -> 254.2 mm, vias 0 -> 2
- net /OUT_FUEL_PUMP: track 0.00 -> 251.7 mm, vias 0 -> 2
- net /GATE_IGN7: track 0.00 -> 224.6 mm, vias 0 -> 1
- net /IN_CAM: track 0.00 -> 183.6 mm, vias 0 -> 2
- net /IN_KNOCK2: track 0.00 -> 181.3 mm, vias 0 -> 1
- net /IN_CLT: track 0.00 -> 176.8 mm, vias 0 -> 1
- net /IN_KNOCK1: track 0.00 -> 174.5 mm, vias 0 -> 1
- net /IN_START_BTN: track 0.00 -> 174.3 mm
- net /CAN_L: track 0.00 -> 170.4 mm, vias 0 -> 1
- net /12V_MR: track 0.00 -> 168.2 mm, vias 0 -> 3
- net /IN_MAF1: track 0.00 -> 165.1 mm, vias 0 -> 3
- net /CAN_H: track 0.00 -> 164.5 mm, vias 0 -> 3
- net /IN_D4: track 0.00 -> 164.0 mm
- net /IN_CRANK+: track 0.00 -> 159.3 mm, vias 0 -> 1
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- added copper zone on B.Cu, net /OUT_IGN1
- added copper zone on F.Cu, net /OUT_IGN7
Other:
- board size 334 x 118 mm -> 350 x 111.3 mm
- board text added: "+5 +5 TPS1_1 TPS1_2 GND GND"
- board text added: "+5 +5 TPS2_1 TPS2_2 GND GND"
- board text added: "+5 AV10 FAN_REL FUEL_PUMP START_BTN D4 D5 GND"
- board text added: "+5 PPS1 PPS2 GND"
- board text added: "- + ETB1"
- board text added: "- + ETB2"
- board text added: "GND GND H- H- Rtrim Ip Vs/Ip VS H+ H+"
- board text added: "IGN1 IGN2 IGN3 IGN4 IGN5 IGN6"
- board text added: "IGN7 IGN8 IGN9 IGN10 IGN11 IGN12"
- board text added: "SWD: R D G C V"
- board text added: "WBO1"
- board text added: "WBO2"
